File: pcb/ErgoDOX.kicad_pcb (KiCad board)
At the start: 2 copper layers, 182.8 x 158.9 mm, 63 parts, among them J1 USB, J2 3.5mm, J3 JMP, J4 JMP, SW0:10 SW0:3, SW0:11 SW0:2, SW0:12 SW0:1, SW0:7 SW0:6, SW0:8 SW0:5, SW0:9 SW0:4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

Commit message: 修正
Gerberファイルを削除。
Teensy2とIOエキスパンダもソケット対応。
Other:
- board text added: "Modified by Hidekingerz"
- board text removed: "Design by Hidekingerz"
